File: lab/lab.kicad_pcb (KiCad board)
At the start: 2 copper layers, 45.7 x 31.8 mm, 33 parts, among them J1 Conn_02x05_Odd_Even, J2 Conn_02x05_Odd_Even, Q1 Q_NPN_EBC, U1 LM324, U2 L78L33_TO92

Commit message: Made a final design.
Parts:
- removed J2: Conn_02x05_Odd_Even, Connector_PinHeader_2.54mm:PinHeader_2x05_P2.54mm_Vertical
- added J3: C?, Connector_PinHeader_2.54mm:PinHeader_1x02_P2.54mm_Vertical, F.Cu at (54.7, 25.5)
- added JP3: MWHAT, Connector_PinHeader_2.54mm:PinHeader_1x03_P2.54mm_Vertical, F.Cu at (49.2, 21.1)
- added JP4: GEN, Connector_PinHeader_2.54mm:PinHeader_2x01_P2.54mm_Vertical, F.Cu at (29.3, 29.8)
- added Q2: Q_NPN_EBC, Package_TO_SOT_THT:TO-92_HandSolder, F.Cu at (24.2, 22.5)
- added Q3: Q_NPN_EBC, Package_TO_SOT_THT:TO-92_HandSolder, F.Cu at (29.6, 20.0)
- added R15: 10K, Resistor_SMD:R_0805_2012Metric_Pad1.15x1.40mm_HandSolder, F.Cu at (24.3, 25.8)
- added R16: 10K, Resistor_SMD:R_0805_2012Metric_Pad1.15x1.40mm_HandSolder, F.Cu at (34.9, 20.8)
- added R17: 1K, Resistor_SMD:R_0805_2012Metric_Pad1.15x1.40mm_HandSolder, F.Cu at (39.3, 20.7)
- added R18: 10K, Resistor_SMD:R_0805_2012Metric_Pad1.15x1.40mm_HandSolder, F.Cu at (29.6, 24.8)
- added R19: 220R, Resistor_SMD:R_0805_2012Metric_Pad1.15x1.40mm_HandSolder, F.Cu at (43.7, 21.1)
- J1: value Conn_02x05_Odd_Even -> FACE
- moved R11 42.2 mm to (25.9, 45.3), turned to 180 degrees
- moved R7 41.1 mm to (62.6, 44.3)
- moved C6 39.5 mm to (25.9, 43.5), turned to 180 degrees
- moved C8 39.2 mm to (59.8, 26.1), turned to 180 degrees
- moved C5 37.2 mm to (60.7, 44.4)
- moved C3 36.5 mm to (56.6, 46.7), turned to 180 degrees
- moved JP2 36.1 mm to (62.2, 40.0), turned to 90 degrees
- moved R6 35.6 mm to (26.8, 39.3), turned to 90 degrees
- moved R5 34.8 mm to (52.9, 44.9), turned to 270 degrees
- moved Q1 33.7 mm to (56.5, 40.1)
- moved RV1 32.3 mm to (22.8, 33.8), turned to 90 degrees
- moved R2 30.1 mm to (58.4, 21.0), turned to 90 degrees
- moved C1 29.9 mm to (31.9, 33.2), turned to 0 degrees
- moved U2 27.8 mm to (52.1, 32.5), turned to 90 degrees
- moved R10 27.2 mm to (32.4, 40.1), turned to 270 degrees
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Connections:
- J1 pad 1: VREF3.3 -> +5V
- J1 pad 10: GNDD -> MEAS
- J1 pad 2: +5V -> CSD1
- J1 pad 3: 3V3 -> SQUARE
- J1 pad 4: +5V -> CSD2
- J1 pad 5: SQUARE -> TRIANGLE
- J1 pad 6: 3V3 -> CMRST
- J1 pad 7: TRIANGLE -> SIN
- J1 pad 8: GNDD -> VREF3.3
- J1 pad 9: SIN -> GNDD
- RV1 pad 1: Net-(C1-Pad1) -> Net-(JP4-Pad2)
Routing:
- net 3V3: track 31.5 -> 92.2 mm, vias 0 -> 2
- net GNDD: track 125.8 -> 69.9 mm, vias 0 -> 2
- net CMEAS: track 0.00 -> 39.1 mm, vias 0 -> 2
- net Net-(R3-Pad1): track 11.9 -> 41.3 mm
- net VREF3.3: track 37.0 -> 22.7 mm
- net Net-(C5-Pad2): track 26.2 -> 12.8 mm
- net Net-(C5-Pad1): track 11.6 -> 24.8 mm
- net SQUARE: track 39.5 -> 27.0 mm
- net +5V: track 67.0 -> 78.5 mm
- net CSD1: track 0.00 -> 9.70 mm
- net Net-(Q3-Pad1): track 0.00 -> 9.59 mm
- net MEAS: track 0.00 -> 8.41 mm
- net TRIANGLE: track 46.8 -> 39.5 mm
- net SIN: track 26.7 -> 33.4 mm, vias 2 -> 0
- net Net-(JP2-Pad2): track 11.3 -> 4.88 mm
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
Commit message: Finalized gerber generation
Parts:
- moved R10 0.47 mm to (32.4, 39.6)
- moved R9 0.26 mm to (47.8, 34.5)
Routing:
- net GNDD: track 69.9 -> 85.9 mm
- net 3V3: track 92.2 -> 106.0 mm
- net SIN: track 33.4 -> 41.7 mm
- net +5V: track 78.5 -> 86.3 mm
- net CMEAS: track 39.1 -> 45.0 mm
- net VREF3.3: track 22.7 -> 25.8 mm
- net Net-(R3-Pad1): track 41.3 -> 43.9 mm
- net Net-(C5-Pad1): track 24.8 -> 27.2 mm
- net SQUARE: track 27.0 -> 29.3 mm
- net Net-(C3-Pad1): track 4.08 -> 5.95 mm
- net Net-(R9-Pad2): track 7.36 -> 8.65 mm
- net Net-(C5-Pad2): track 12.8 -> 14.1 mm
- net Net-(Q3-Pad1): track 9.59 -> 10.5 mm
- net CSD1: track 9.70 -> 10.5 mm
- net TRIANGLE: track 39.5 -> 40.3 mm
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- added copper zone on F.Cu, net +5V
- added copper zone on F.Cu, net 3V3
- added copper zone on F.Cu, net GNDD
- added copper zone on F.Cu, net Net-(C3-Pad1)
- added copper zone on F.Cu, net Net-(C5-Pad1)
- added copper zone on F.Cu, net Net-(JP2-Pad2)
Other:
- net class Default: via_dia 0.8 -> 2; via_drill 0.4 -> 1
