File: lab/lab.kicad_pcb (KiCad board)
At the start: 2 copper layers, 45.7 x 31.8 mm, 42 parts, among them J1 FACE, J3 C?, Q1 Q_NPN_EBC, Q2 Q_NPN_EBC, Q3 Q_NPN_EBC, U1 LM324, U2 L78L33_TO92

Commit message: The current state.
Routing:
- net +5V: track 173.8 -> 171.5 mm
Changed lines of the file:
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@@
     (thickness 1.6)
     (drawings 6)
-    (tracks 838)
+    (tracks 836)
     (zones 0)
     (modules 42)
@@
   )
   (setup
-    (last_trace_width 1)
+    (last_trace_width 0.35)
     (user_trace_width 0.25)
     (user_trace_width 0.5)
@@
   (segment (start 21.672326 28.702) (end 24.638 28.702) (width 0.5) (layer F.Cu) (net 3))
   (segment (start 24.638 28.702) (end 25.4 29.464) (width 0.5) (layer F.Cu) (net 3))
-  (segment (start 38.354 48.768) (end 37.7776 48.1916) (width 0.5) (layer F.Cu) (net 3))
   (segment (start 37.7776 48.1916) (end 37.7776 45.5375) (width 0.5) (layer F.Cu) (net 3))
   (segment (start 64.19499 40.06499) (end 64.19499 48.768) (width 0.5) (layer F.Cu) (net 3))
@@
   (segment (start 38.864883 47.7375) (end 39.832373 48.70499) (width 1) (layer F.Cu) (net 3))
   (segment (start 37.7776 47.7375) (end 38.864883 47.7375) (width 1) (layer F.Cu) (net 3))
-  (segment (start 39.832373 48.70499) (end 38.354 48.768) (width 0.5) (layer F.Cu) (net 3))
   (segment (start 54.8523 46.0493) (end 55.0523 46.0493) (width 0.35) (layer F.Cu) (net 4) (status 30))
   (segment (start 55.0523 46.0493) (end 55.3001 46.0493) (width 0.35) (layer F.Cu) (net 4) (status 30))
